File: nkc_pcb/nkc_pcb.kicad_sch (KiCad schematic)
At the start: 0 parts

Commit message: add resources, 2 components
Parts:
- added A1: RaspberryPi_Pico, Module_RaspberryPi_Pico:RaspberryPi_Pico_Common, symbol MCU_Module_RaspberryPi_Pico:RaspberryPi_Pico
- added U1: CD74HC4067M, Package_SO:SOIC-24W_7.5x15.4mm_P1.27mm, symbol 74xx:CD74HC4067M
Connections:
- new net: A1.36 (3V3), U1.24 (VCC)
- new net GND: A1.13 (GND), A1.18 (GND), A1.23 (GND), A1.28 (GND), A1.3 (GND), A1.38 (GND), A1.8 (GND), U1.12 (GND)
Other:
- company: (none) -> UF Audio Engineering Society
- title: (none) -> Necroknobicon
